File: Electronica/El_Empujon/El_Empujon.kicad_sch (KiCad schematic)
At the start: 0 parts

Commit message: Actualizacion del esquematico , adicion de los datasheet a las documentacion e inicio de la PCB
Other:
- added sheet Alimentacion (Alimentacion.kicad_sch)
- added sheet BTS7960 (Potencia y Motores.kicad_sch)
- added sheet Esp32 (micro.kicad_sch)
- added sheet VL53L0X y TCRT5000 (Deteccion.kicad_sch)
- note added: "El empujon"

Commit message: Generacion del STEP, finalizacion del esquematico y de la PCB, generacion de los archivos de manufactura de la PCB, Pedido de la PCB y actualizacion del Presupuesto.
Connections:
- no-connect marks 0 -> 22
Other:
- sheet Alimentacion ports: added 3.3V; removed none
- sheet BTS7960 ports: added 3.3V, 5V; removed VCC
