File: Electronica/El_Empujon/Potencia y Motores.kicad_sch (KiCad schematic)
At the start: 4 parts, among them J5 Conn_01x08_Socket, J6 Conn_01x04_Socket, J7 Conn_01x08_Socket, J8 Conn_01x04_Socket

Commit message: Generacion del STEP, finalizacion del esquematico y de la PCB, generacion de los archivos de manufactura de la PCB, Pedido de la PCB y actualizacion del Presupuesto.
Connections:
- net VCC renamed 3.3V
- net 3.3V: no longer J5.7 (Pin_7), J7.7 (Pin_7)
- new net 5V: J5.7 (Pin_7), J7.7 (Pin_7)
Other:
- note added: "Drivers"
- note added: "Encoder del motor"
- note removed: "Encoder"
- note removed: "Motores"
Changed lines of the file:
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@@
 		)
 	)
-	(text "Encoder"
+	(text "Encoder del motor"
 		(exclude_from_sim no)
 		(at 87.376 101.346 0)
@@
 		)
 	)
-	(text "Motores"
+	(text "Drivers"
 		(exclude_from_sim no)
 		(at 83.566 43.942 0)
@@
 		)
 	)
-	(hierarchical_label "VCC"
+	(hierarchical_label "5V"
 		(shape input)
 		(at 49.53 69.85 180)
@@
 		)
 	)
-	(hierarchical_label "VCC"
+	(hierarchical_label "3.3V"
 		(shape input)
 		(at 107.95 121.92 180)
@@
 		)
 	)
-	(hierarchical_label "VCC"
+	(hierarchical_label "3.3V"
 		(shape input)
 		(at 54.61 121.92 180)
@@
 		)
 	)
-	(hierarchical_label "VCC"
+	(hierarchical_label "5V"
 		(shape input)
 		(at 102.87 71.12 180)
