File: Electronica/El_Empujon/micro.kicad_sch (KiCad schematic)
At the start: 2 parts, among them J3 Conn_01x19_Socket, J4 Conn_01x19_Socket

Commit message: Generacion del STEP, finalizacion del esquematico y de la PCB, generacion de los archivos de manufactura de la PCB, Pedido de la PCB y actualizacion del Presupuesto.
Changed lines of the file:
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@@
 	)
 	(hierarchical_label "3.3V"
-		(shape input)
+		(shape output)
 		(at 45.72 72.39 180)
 		(effects
